File: HVAC_STM32F7_PCB/_autosave-HVAC_STM32F7_PCB.kicad_pcb (KiCad board)
At the start: 4 copper layers, 91 parts, among them J1 DC_Jack_5.5x2.1mm, J10 OUT_Signal_connector, J11 OUT_Signal_connector, J12 OUT_Signal_connector, J13 OUT_Signal_connector, J14 Signal_connector, J15 Signal_connector, J16 Signal_connector, J17 Signal_connector, J2 Signal_connector, J3 Signal_connector, J4 Signal_connector, J5 Signal_connector, J6 OUT_Signal_connector, J7 OUT_Signal_connector, J8 OUT_Signal_connector, J9 OUT_Signal_connector, Q1 IRLML9301, U1 LM2596S-5, U2 LM2596S-3.3, U5 TLV9304xPW, U6 TLV9304xPW, U7 ADS8688

Commit message: ADD: working first draft compilation of documentation, PCB project playing around
Parts:
- moved C10 150.8 mm to (221.8, 35.8)
- moved C11 150.8 mm to (221.8, 38.8)
- moved C11X7R1 150.8 mm to (221.8, 47.8)
- moved C12 150.8 mm to (221.8, 41.8)
- moved C13 150.8 mm to (221.8, 44.8)
- moved C9 150.8 mm to (221.8, 32.8)
- moved J14 150.8 mm to (205.4, 73.9)
- moved J15 150.8 mm to (205.4, 83.3)
- moved J16 150.8 mm to (205.4, 92.6)
- moved J17 150.8 mm to (205.4, 101.9)
- moved J2 150.8 mm to (205.4, 36.6)
- moved J3 150.8 mm to (205.4, 45.9)
- moved J4 150.8 mm to (205.4, 55.3)
- moved J5 150.8 mm to (205.4, 64.6)
- moved R1 150.8 mm to (221.8, 62.2)
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